File: cubesat-panel.kicad_pcb (KiCad board)
At the start: 2 copper layers, 80 x 95 mm, 18 parts, among them J1 CONN-TAB, J10 MOLEX_FFC-14, J2 CONN-TAB, J3 CONN-TAB, J4 CONN-TAB, J5 CONN-TAB, J6 CONN-TAB, J7 CONN-TAB, J8 CONN-TAB, J9 MOLEX_FFC-14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

Commit message: PV layout optimized for routing
Parts:
- moved J8 91.4 mm to (168.0, 236.0)
- moved J3 90.4 mm to (152.0, 147.0)
- moved J6 89.1 mm to (172.0, 236.0)
- moved J1 89.0 mm to (148.0, 147.0)
- moved P2 57.3 mm to (140.0, 212.0)
- moved P3 57.3 mm to (180.0, 171.0)
- moved J4 21.0 mm to (152.0, 236.0)
- moved J7 16.0 mm to (168.0, 147.0)
- moved J2 4.00 mm to (148.0, 236.0)
- moved J5 1.00 mm to (172.0, 147.0)
- turned P1 to 0 degrees
- turned P4 to 0 degrees
Connections:
- J4 pad 1: Net-(J4-Pad1) -> Net-(J3-Pad1)
- J8 pad 1: Net-(J8-Pad1) -> Net-(J7-Pad1)
- P1 pad 1: Net-(P1-Pad1) -> Net-(J1-Pad1)
- P2 pad 1: Net-(P2-Pad1) -> Net-(P1-Pad2)
- P2 pad 2: Net-(P2-Pad2) -> Net-(J2-Pad1)
- P3 pad 1: Net-(P3-Pad1) -> Net-(J5-Pad1)
- P4 pad 1: Net-(P4-Pad1) -> Net-(P3-Pad2)
- P4 pad 2: Net-(P4-Pad2) -> Net-(J6-Pad1)

Commit message: Added drawing of access panel
Other:
- board text added: "+Z"
- board text added: "Access Panel"
- board text added: "Cabling"

Commit message: Modified to single panel. To reduce integration complexity the formerly 3 panel configuration was changed to a single 300mm x 80mm board per side.
Parts:
- added C1: 0.1uF, Capacitors_SMD:C_0402, F.Cu at (125.2, 39.8)
- added C2: 0.1uF, Capacitors_SMD:C_0402, F.Cu at (125.6, 187.2)
- added C3: 0.1uF, Capacitors_SMD:C_0402, F.Cu at (125.6, 329.4)
- added C4: 0.1uF, Capacitors_SMD:C_0402, F.Cu at (193.6, 47.0)
- added C5: 0.1uF, Capacitors_SMD:C_0402, F.Cu at (194.4, 192.6)
- added C6: 0.1uF, Capacitors_SMD:C_0402, F.Cu at (194.0, 335.6)
- added D5: D_Photo, SFUSat:SFH2430, F.Cu at (196.8, 189.4)
- added D6: D_Photo, SFUSat:SFH2430, F.Cu at (196.4, 332.4)
- added P10: JSLINTER, SFUSat:JSLINTER-39x26, F.Cu at (180.0, 219.0)
- added P11: JSLINTER, SFUSat:JSLINTER-39x26, F.Cu at (180.0, 260.0)
- added P12: JSLINTER, SFUSat:JSLINTER-39x26, F.Cu at (180.0, 301.0)
- added P5: JSLINTER, SFUSat:JSLINTER-39x26, F.Cu at (140.0, 260.0)
- added P6: JSLINTER, SFUSat:JSLINTER-39x26, F.Cu at (140.0, 301.0)
- added P7: JSLINTER, SFUSat:JSLINTER-39x26, F.Cu at (180.0, 69.0)
- added P8: JSLINTER, SFUSat:JSLINTER-39x26, F.Cu at (180.0, 110.0)
- added P9: JSLINTER, SFUSat:JSLINTER-39x26, F.Cu at (180.0, 164.0)
- added R1: R, Resistors_SMD:R_0402, F.Cu at (131.0, 43.2)
- added R10: R, Resistors_SMD:R_0402, F.Cu at (187.6, 189.6)
- added R11: R, Resistors_SMD:R_0402, F.Cu at (188.4, 332.6)
- added R12: R, Resistors_SMD:R_0402, F.Cu at (187.2, 332.6)
- added R2: R, Resistors_SMD:R_0402, F.Cu at (132.2, 43.2)
- added R3: R, Resistors_SMD:R_0402, F.Cu at (131.2, 190.0)
- added R4: R, Resistors_SMD:R_0402, F.Cu at (132.4, 190.0)
- added R5: R, Resistors_SMD:R_0402, F.Cu at (131.2, 332.2)
- added R6: R, Resistors_SMD:R_0402, F.Cu at (132.4, 332.2)
- added R7: R, Resistors_SMD:R_0402, F.Cu at (188.0, 44.0)
- added R8: R, Resistors_SMD:R_0402, F.Cu at (186.8, 44.0)
- added R9: R, Resistors_SMD:R_0402, F.Cu at (188.8, 189.6)
- added U1: OPA380, SFUSat:VSSOP_8, F.Cu at (128.0, 43.2)
- added U2: OPA380, SFUSat:VSSOP_8, F.Cu at (128.4, 190.0)
- added U3: OPA380, SFUSat:VSSOP_8, F.Cu at (128.4, 332.2)
- added U4: OPA380, SFUSat:VSSOP_8, F.Cu at (190.8, 44.0)
- added U5: OPA380, SFUSat:VSSOP_8, F.Cu at (191.6, 189.6)
- added U6: OPA380, SFUSat:VSSOP_8, F.Cu at (191.2, 332.4)
- moved D3 197.6 mm to (123.4, 332.6), turned to 270 degrees
- moved D1 192.8 mm to (123.0, 43.2), turned to 270 degrees
- moved D4 125.6 mm to (196.2, 43.8), turned to 90 degrees
- moved J1 106.0 mm to (148.0, 41.0)
- moved J3 106.0 mm to (152.0, 41.0)
- moved J5 106.0 mm to (172.0, 41.0)
- moved J7 106.0 mm to (168.0, 41.0)
- moved J9 106.0 mm to (160.0, 41.0)
- moved P1 102.0 mm to (140.0, 69.0)
- moved P2 102.0 mm to (140.0, 110.0)
- moved J10 99.0 mm to (160.0, 335.0)
- moved J2 99.0 mm to (148.0, 335.0)
- moved J4 99.0 mm to (152.0, 335.0)
- moved J6 99.0 mm to (172.0, 335.0)
- moved J8 99.0 mm to (168.0, 335.0)
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Connections:
- D1 pad 2: Net-(D1-Pad2) -> GND
- D2 pad 2: Net-(D2-Pad2) -> GND
- D3 pad 2: Net-(D3-Pad2) -> GND
- D4 pad 2: Net-(D4-Pad2) -> GND
- J10 pad SHLD: Net-(J10-PadSHLD) -> GND
- J9 pad SHLD: Net-(J9-PadSHLD) -> GND
- P2 pad 2: Net-(J2-Pad1) -> Net-(P2-Pad2)
- P3 pad 1: Net-(J5-Pad1) -> Net-(P2-Pad2)
- P4 pad 2: Net-(J6-Pad1) -> Net-(P4-Pad2)
Other:
- board size 80 x 95 mm -> 80 x 300 mm
- board text added: "Access Panel Geometry Per 2018-02-01 OBC Board"
- board text added: "D0"
- board text added: "D1"
- board text added: "D2"
- board text added: "D3"
- board text added: "D4"
- board text added: "D5"
- board text added: "Photodiode Layout"
- board text removed: "CubeSat Outer Panels"

Commit message: Layed out components. General layout of sun sensor sub system, PV, mounting hole, connectors, access panel cutout is complete. Yet to finalize ribbon cable signal layout and PV orientation.
Parts:
- added J11: PC104PTH, SFUSat:PTH-2.0mm, F.Cu at (140.0, 42.0)
- added J12: PC104PTH, SFUSat:PTH-2.0mm, F.Cu at (123.0, 144.0)
- added J13: PC104PTH, SFUSat:PTH-2.0mm, F.Cu at (123.0, 236.0)
- added J14: PC104PTH, SFUSat:PTH-2.0mm, F.Cu at (139.0, 328.0)
- added J15: PC104PTH, SFUSat:PTH-2.0mm, F.Cu at (160.0, 65.0)
- added J16: PC104PTH, SFUSat:PTH-2.0mm, F.Cu at (160.0, 144.0)
- added J17: PC104PTH, SFUSat:PTH-2.0mm, F.Cu at (160.0, 237.0)
- added J18: PC104PTH, SFUSat:PTH-2.0mm, F.Cu at (160.0, 316.0)
- added J19: PC104PTH, SFUSat:PTH-2.0mm, F.Cu at (179.0, 42.0)
- added J20: PC104PTH, SFUSat:PTH-2.0mm, F.Cu at (197.0, 144.0)
- added J21: PC104PTH, SFUSat:PTH-2.0mm, F.Cu at (197.0, 236.0)
- added J22: PC104PTH, SFUSat:PTH-2.0mm, F.Cu at (180.0, 328.0)
- moved P1 13.0 mm to (140.0, 82.0)
- moved P2 13.0 mm to (140.0, 123.0)
- moved P7 13.0 mm to (180.0, 82.0)
- moved P8 13.0 mm to (180.0, 123.0)
- moved C3 6.00 mm to (125.6, 323.4)
- moved C6 6.00 mm to (194.0, 329.6)
- moved D3 6.00 mm to (123.4, 326.6)
- moved D6 6.00 mm to (196.4, 326.4)
- moved J10 6.00 mm to (160.0, 329.0)
- moved J2 6.00 mm to (148.0, 329.0)
- moved J4 6.00 mm to (152.0, 329.0)
- moved J6 6.00 mm to (172.0, 329.0)
- moved J8 6.00 mm to (168.0, 329.0)
- moved R11 6.00 mm to (188.4, 326.6)
- moved R12 6.00 mm to (187.2, 326.6)
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Other:
- board size 80 x 300 mm -> 80 x 294 mm
- board text added: "Cable Entry Slot"
- board text added: "Umbilical is only present on the -X face"
- board text removed: "Slot Dimentions are provisional"

Commit message: generated 3d model
Parts:
- moved J9 3.40 mm to (160.0, 44.4), turned to 180 degrees
- moved J10 3.40 mm to (160.0, 325.6), turned to 0 degrees
Other:
- outline, holes or cut-outs redrawn

Commit message: initial routing
Parts:
- removed J3, J4, J7, J8: CONN-TAB, SFUSat:CONN_TAB
- R1, R11, R3, R5, R7, R9: value R -> 2K2
- R10, R12, R2, R4, R6, R8: value R -> DNP
- moved J5 288.0 mm to (168.0, 329.0)
- moved J1 288.0 mm to (148.0, 329.0)
- moved J9 280.1 mm to (160.0, 324.5), turned to 0 degrees
- moved J10 278.6 mm to (160.0, 47.0), turned to 180 degrees
- moved C1 7.96 mm to (132.4, 43.2), turned to 270 degrees
- moved C4 7.80 mm to (186.4, 44.0), turned to 90 degrees
- moved C2 7.73 mm to (132.8, 190.0), turned to 270 degrees
- moved C5 7.62 mm to (187.4, 189.6), turned to 90 degrees
- moved C6 7.62 mm to (187.0, 326.6), turned to 90 degrees
- moved C3 7.54 mm to (132.6, 326.2), turned to 270 degrees
- moved R6 5.28 mm to (129.2, 322.0), turned to 0 degrees
- moved J2 4.00 mm to (152.0, 329.0)
- moved R2 2.78 mm to (130.8, 40.8), turned to 90 degrees
- moved R10 2.51 mm to (188.8, 191.8), turned to 270 degrees
- moved R12 2.51 mm to (188.4, 328.8), turned to 270 degrees
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Connections:
- net Net-(J1-Pad1) renamed /PV1+
- net Net-(J2-Pad1) renamed /PV1-
- net Net-(J5-Pad1) renamed /PV2+
- net Net-(J6-Pad1) renamed /PV2-
- C1 pad 1: /Sun_Sensor_0/VCC -> /D0
- C1 pad 2: GND -> Net-(C1-Pad2)
- C2 pad 1: /Sun_Sensor_0/VCC -> /D1
- C2 pad 2: GND -> Net-(C2-Pad2)
- C3 pad 1: /Sun_Sensor_0/VCC -> /D2
- C3 pad 2: GND -> Net-(C3-Pad2)
- C4 pad 1: /Sun_Sensor_0/VCC -> /D3
- C4 pad 2: GND -> Net-(C4-Pad2)
- C5 pad 1: /Sun_Sensor_0/VCC -> /D4
- C5 pad 2: GND -> Net-(C5-Pad2)
- C6 pad 1: /Sun_Sensor_0/VCC -> /D5
- C6 pad 2: GND -> Net-(C6-Pad2)
- D1 pad 1: Net-(D1-Pad1) -> Net-(C1-Pad2)
- D2 pad 1: Net-(D2-Pad1) -> Net-(C2-Pad2)
- D3 pad 1: Net-(D3-Pad1) -> Net-(C3-Pad2)
- D4 pad 1: Net-(D4-Pad1) -> Net-(C4-Pad2)
- D5 pad 1: Net-(D5-Pad1) -> Net-(C5-Pad2)
- D6 pad 1: Net-(D6-Pad1) -> Net-(C6-Pad2)
- J10 pad 1: Net-(J10-Pad1) -> /3V3
- J10 pad 13: Net-(J10-Pad13) -> GND
- J10 pad 14: Net-(J10-Pad14) -> /3V3
- J10 pad 2: Net-(J10-Pad2) -> GND
- J10 pad 6: Net-(J10-Pad6) -> /D6
- J10 pad 7: Net-(J10-Pad7) -> /D7
- J10 pad 8: Net-(J10-Pad8) -> /D8
- J10 pad 9: Net-(J10-Pad9) -> /D9
- J9 pad 1: Net-(J9-Pad1) -> /3V3
- J9 pad 10: Net-(J9-Pad10) -> /D3
- J9 pad 11: Net-(J9-Pad11) -> /D4
- J9 pad 12: Net-(J9-Pad12) -> /D5
- J9 pad 13: Net-(J9-Pad13) -> GND
- J9 pad 14: Net-(J9-Pad14) -> /3V3
- J9 pad 2: Net-(J9-Pad2) -> GND
- J9 pad 3: Net-(J9-Pad3) -> /D2
- J9 pad 4: Net-(J9-Pad4) -> /D1
- J9 pad 5: Net-(J9-Pad5) -> /D0
- J9 pad 6: Net-(J9-Pad6) -> /D6
- J9 pad 7: Net-(J9-Pad7) -> /D7
- J9 pad 8: Net-(J9-Pad8) -> /D8
- J9 pad 9: Net-(J9-Pad9) -> /D9
- R1 pad 2: Net-(D1-Pad1) -> Net-(C1-Pad2)
- R11 pad 2: Net-(D6-Pad1) -> Net-(C6-Pad2)
- R3 pad 2: Net-(D2-Pad1) -> Net-(C2-Pad2)
- R5 pad 2: Net-(D3-Pad1) -> Net-(C3-Pad2)
- R7 pad 2: Net-(D4-Pad1) -> Net-(C4-Pad2)
- R9 pad 2: Net-(D5-Pad1) -> Net-(C5-Pad2)
- U1 pad 2: Net-(D1-Pad1) -> Net-(C1-Pad2)
- U2 pad 2: Net-(D2-Pad1) -> Net-(C2-Pad2)
- U3 pad 2: Net-(D3-Pad1) -> Net-(C3-Pad2)
- U4 pad 2: Net-(D4-Pad1) -> Net-(C4-Pad2)
- U5 pad 2: Net-(D5-Pad1) -> Net-(C5-Pad2)
- U6 pad 2: Net-(D6-Pad1) -> Net-(C6-Pad2)
Routing:
- net /PV2+: track 0.00 -> 258.2 mm
- net /PV1+: track 0.00 -> 250.5 mm
- net /Sun_Sensor_0/VCC: track 0.00 -> 198.0 mm, vias 0 -> 4
- net Net-(P3-Pad2): track 0.00 -> 66.9 mm
- net Net-(P10-Pad1): track 0.00 -> 52.0 mm
- net Net-(P10-Pad2): track 0.00 -> 45.1 mm
- net Net-(P8-Pad2): track 0.00 -> 44.3 mm
- net /PV2-: track 0.00 -> 41.1 mm
- net Net-(P7-Pad2): track 0.00 -> 41.0 mm
- net Net-(P5-Pad2): track 0.00 -> 41.0 mm
- net Net-(P4-Pad2): track 0.00 -> 41.0 mm
- net Net-(P2-Pad2): track 0.00 -> 41.0 mm
- net Net-(P11-Pad2): track 0.00 -> 41.0 mm
- net Net-(P1-Pad2): track 0.00 -> 41.0 mm
- net /PV1-: track 0.00 -> 32.2 mm
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- added copper zone on B.Cu, net GND
Other:
- outline, holes or cut-outs redrawn
- net class PV added: clearance 0.4, trace_width 2.2, via_dia 0.6, via_drill 0.4

Commit message: added new access cutout
Parts:
- added REF**: NPTH-1mm, SFUSat:NPTH-1mm, F.Cu at (166.0, 43.0)
- added REF**: NPTH-1mm, SFUSat:NPTH-1mm, F.Cu at (154.0, 43.0)
- added REF**: NPTH-1mm, SFUSat:NPTH-1mm, F.Cu at (154.0, 330.0)
- added REF**: NPTH-1mm, SFUSat:NPTH-1mm, F.Cu at (166.0, 330.0)
- moved R2 37.6 mm to (125.6, 78.0), turned to 270 degrees
- moved C1 36.9 mm to (123.4, 79.0), turned to 180 degrees
- moved C4 36.6 mm to (196.2, 79.2), turned to 180 degrees
- moved R1 35.2 mm to (123.4, 77.6), turned to 180 degrees
- moved R7 34.6 mm to (196.2, 77.7), turned to 180 degrees
- moved R8 33.5 mm to (198.2, 78.0)
- moved U1 31.7 mm to (123.4, 74.6), turned to 270 degrees
- moved U4 31.3 mm to (196.2, 74.8), turned to 270 degrees
- moved P10 27.0 mm to (180.0, 189.0)
- moved P11 27.0 mm to (180.0, 230.0)
- moved P12 27.0 mm to (180.0, 271.0)
- moved P4 27.0 mm to (140.0, 189.0)
- moved P5 27.0 mm to (140.0, 230.0)
- moved P6 27.0 mm to (140.0, 271.0)
- moved D1 25.0 mm to (123.4, 68.2)
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Connections:
- net /D9 renamed /DA
- C1 pad 1: /D0 -> /D6
- C2 pad 1: /D1 -> /D7
- C3 pad 1: /D2 -> /D8
- C5 pad 1: /D4 -> /D2
- C6 pad 1: /D5 -> /D1
- J10 pad 6: /D6 -> /DB
- J10 pad 7: /D7 -> GND
- J10 pad 8: /D8 -> GND
- J11 pad 1: Net-(J11-Pad1) -> GND
- J12 pad 1: Net-(J12-Pad1) -> GND
- J13 pad 1: Net-(J13-Pad1) -> GND
- J14 pad 1: Net-(J14-Pad1) -> GND
- J15 pad 1: Net-(J15-Pad1) -> GND
- J16 pad 1: Net-(J16-Pad1) -> GND
- J17 pad 1: Net-(J17-Pad1) -> GND
- J18 pad 1: Net-(J18-Pad1) -> GND
- J19 pad 1: Net-(J19-Pad1) -> GND
- J20 pad 1: Net-(J20-Pad1) -> GND
- J21 pad 1: Net-(J21-Pad1) -> GND
- J22 pad 1: Net-(J22-Pad1) -> GND
- J9 pad 11: /D4 -> /D2
- J9 pad 12: /D5 -> /D1
- J9 pad 3: /D2 -> /D8
- J9 pad 4: /D1 -> /D7
- J9 pad 5: /D0 -> /D6
- J9 pad 6: /D6 -> /DB
- J9 pad 7: /D7 -> GND
- J9 pad 8: /D8 -> GND
- R1 pad 1: /D0 -> /D6
- R10 pad 1: /D4 -> /D2
- R11 pad 1: /D5 -> /D1
- R12 pad 1: /D5 -> /D1
- R2 pad 1: /D0 -> /D6
- R3 pad 1: /D1 -> /D7
- R4 pad 1: /D1 -> /D7
- R5 pad 1: /D2 -> /D8
- R6 pad 1: /D2 -> /D8
- R9 pad 1: /D4 -> /D2
- U1 pad 6: /D0 -> /D6
- U2 pad 6: /D1 -> /D7
- U3 pad 6: /D2 -> /D8
- U5 pad 6: /D4 -> /D2
- U6 pad 6: /D5 -> /D1
Routing:
- net /PV2+: track 258.2 -> 0.00 mm
- net /PV1+: track 250.5 -> 0.00 mm
- net /Sun_Sensor_0/VCC: track 198.0 -> 1.36 mm, vias 4 -> 1
- net (no net): track 0.00 -> 125.7 mm
- net Net-(P3-Pad2): track 66.9 -> 0.00 mm
- net Net-(P10-Pad1): track 52.0 -> 0.00 mm
- net Net-(P10-Pad2): track 45.1 -> 0.00 mm
- net Net-(P8-Pad2): track 44.3 -> 0.00 mm
- net /PV2-: track 41.1 -> 0.00 mm
- net Net-(P7-Pad2): track 41.0 -> 0.00 mm
- net Net-(P5-Pad2): track 41.0 -> 0.00 mm
- net Net-(P4-Pad2): track 41.0 -> 0.00 mm
- net Net-(P2-Pad2): track 41.0 -> 0.00 mm
- net Net-(P11-Pad2): track 41.0 -> 0.00 mm
- net Net-(P1-Pad2): track 41.0 -> 0.00 mm
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Other:
- outline, holes or cut-outs redrawn
- rule pad_to_mask_clearance: 0.2 -> 0.05
- board text added: "D6"
- board text added: "D7"
- board text added: "D8"

Commit message: modified access panel geometry for new DC jacks, RBF, and Jtag, usb
Parts:
- added REF**: NPTH-1mm, SFUSat:NPTH-1mm, F.Cu at (154.0, 321.5)
- added REF**: NPTH-1mm, SFUSat:NPTH-1mm, F.Cu at (166.0, 321.5)
- moved C2 22.8 mm to (123.4, 178.6), turned to 0 degrees
- moved R4 20.9 mm to (121.2, 179.8), turned to 90 degrees
- moved R3 19.6 mm to (123.4, 180.2), turned to 0 degrees
- moved P12 16.0 mm to (180.0, 287.0)
- moved P6 16.0 mm to (140.0, 287.0)
- moved C6 15.5 mm to (195.4, 310.3), turned to 0 degrees
- moved R12 14.1 mm to (193.6, 311.5), turned to 90 degrees
- moved U2 14.0 mm to (123.4, 183.0), turned to 90 degrees
- moved R11 13.5 mm to (195.4, 311.7), turned to 0 degrees
- moved P11 13.0 mm to (180.0, 243.0)
- moved P5 13.0 mm to (140.0, 243.0)
- moved J9 12.8 mm to (160.0, 310.7)
- moved P10 11.0 mm to (180.0, 200.0)
- moved P4 11.0 mm to (140.0, 200.0)
- moved U6 9.55 mm to (195.6, 314.5), turned to 90 degrees
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Other:
- outline, holes or cut-outs redrawn
