File: cubesat-panel.kicad_pcb (KiCad board)
At the start: 2 copper layers, 80 x 294 mm, 66 parts, among them J1 CONN-TAB, J10 MOLEX_FFC-14, J11 PC104PTH, J12 PC104PTH, J13 PC104PTH, J14 PC104PTH, J15 PC104PTH, J16 PC104PTH, J17 PC104PTH, J18 PC104PTH, J19 PC104PTH, J2 CONN-TAB, J20 PC104PTH, J21 PC104PTH, J22 PC104PTH, J5 CONN-TAB, J6 CONN-TAB, J9 MOLEX_FFC-14, P1 JSLINTER, P10 JSLINTER, P11 JSLINTER, P12 JSLINTER, P2 JSLINTER, P3 JSLINTER, P4 JSLINTER, P5 JSLINTER, P6 JSLINTER, P7 JSLINTER, P8 JSLINTER, P9 JSLINTER, U1 OPA380, U2 OPA380, U3 OPA380, U4 OPA380, U5 OPA380, U6 OPA380

Commit message: layout complete
Parts:
- moved C3 23.9 mm to (138.8, 328.6), turned to 270 degrees
- moved R6 22.4 mm to (137.9, 326.5), turned to 0 degrees
- moved C6 22.0 mm to (183.5, 328.8), turned to 90 degrees
- moved R5 21.9 mm to (137.4, 328.6), turned to 270 degrees
- moved R12 21.1 mm to (184.7, 330.6), turned to 180 degrees
- moved R11 20.1 mm to (184.9, 328.8), turned to 90 degrees
- moved U3 17.9 mm to (134.6, 328.6), turned to 0 degrees
- moved U6 16.2 mm to (187.7, 328.6), turned to 180 degrees
- moved D3 8.35 mm to (128.3, 327.8), turned to 270 degrees
- moved D6 7.69 mm to (192.2, 327.8), turned to 270 degrees
Connections:
- U1 pad 7: /Sun_Sensor_0/VCC -> /3V3
- U2 pad 7: /Sun_Sensor_0/VCC -> /3V3
- U3 pad 7: /Sun_Sensor_0/VCC -> /3V3
- U4 pad 7: /Sun_Sensor_0/VCC -> /3V3
- U5 pad 7: /Sun_Sensor_0/VCC -> /3V3
- U6 pad 7: /Sun_Sensor_0/VCC -> /3V3
Routing:
- net /3V3: track 0.00 -> 511.9 mm, vias 0 -> 13
- net /PV1+: track 0.00 -> 301.0 mm
- net /PV2+: track 0.00 -> 295.5 mm
- net /DA: track 0.00 -> 280.2 mm, vias 0 -> 2
- net /DB: track 0.00 -> 279.0 mm, vias 0 -> 2
- net /D6: track 7.16 -> 255.1 mm, vias 0 -> 2
- net /D3: track 6.98 -> 253.3 mm, vias 0 -> 2
- net /D2: track 6.78 -> 153.1 mm, vias 0 -> 2
- net /D7: track 7.18 -> 151.7 mm, vias 0 -> 2
- net (no net): track 125.7 -> 0.00 mm
- net Net-(P7-Pad2): track 0.00 -> 74.3 mm
- net /PV2-: track 0.00 -> 62.8 mm
- net Net-(P1-Pad2): track 0.00 -> 58.6 mm
- net Net-(P3-Pad2): track 0.00 -> 49.6 mm
- net Net-(P8-Pad2): track 0.00 -> 46.0 mm
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Other:
- board size 80 x 294 mm -> 80 x 295.7 mm

Commit message: optimized silkscreen visibility, generated gerbers
Parts:
- added G***: LOGO, SFUSat:SFUSat_15mm_2, F.Cu at (125.7, 313.9)
Other:
- board text added: "SFU Satellite Design Team Panel Rev. 1"

Commit message: moved FFC position in accordance to PowerSystems Doc
Parts:
- added J3: MOLEX_FFC-14, SFUSat:MOLEX_FFC-14, F.Cu at (160.0, 316.2)
- moved J10 4.14 mm to (160.0, 50.2)
- moved J9 1.31 mm to (160.0, 312.0)
- moved REF** 1.00 mm to (166.0, 43.5)
- moved REF** 1.00 mm to (154.0, 43.5)
Routing:
- net GND: track 39.8 -> 54.2 mm, vias 28 -> 34
- net /DB: track 279.0 -> 288.6 mm
- net /DA: track 280.2 -> 289.8 mm
- net /D7: track 151.7 -> 157.2 mm
- net /D6: track 255.1 -> 260.6 mm
- net /D2: track 153.1 -> 158.6 mm
- net /D3: track 253.3 -> 258.7 mm
- net /3V3: track 511.9 -> 514.5 mm, vias 13 -> 14
- net /D1: track 40.8 -> 39.5 mm
- net /D8: track 36.6 -> 36.0 mm
Other:
- board text added: "X"
- board text added: "Y"

Commit message: improved silkscreen labeling
Other:
- board size 80 x 295.7 mm -> 80 x 294 mm
- board text added: "+z"
- board text added: "-z"
- board text added: "PV+"
- board text added: "PV-"
