File: cubesat-panel.kicad_pcb (KiCad board)
At the start: 2 copper layers, 80 x 294 mm, 68 parts, among them J1 CONN-TAB, J10 MOLEX_FFC-14, J11 PC104PTH, J12 PC104PTH, J13 PC104PTH, J14 PC104PTH, J15 PC104PTH, J16 PC104PTH, J17 PC104PTH, J18 PC104PTH, J19 PC104PTH, J2 CONN-TAB, J20 PC104PTH, J21 PC104PTH, J22 PC104PTH, J3 MOLEX_FFC-14, J5 CONN-TAB, J6 CONN-TAB, J9 MOLEX_FFC-14, P1 JSLINTER, P10 JSLINTER, P11 JSLINTER, P12 JSLINTER, P2 JSLINTER, P3 JSLINTER, P4 JSLINTER, P5 JSLINTER, P6 JSLINTER, P7 JSLINTER, P8 JSLINTER, P9 JSLINTER, U1 OPA380, U2 OPA380, U3 OPA380, U4 OPA380, U5 OPA380, U6 OPA380

Commit message: solder mask fixed to conform to min 150um webbing requirement
Other:
- rule pad_to_mask_clearance: 0.05 -> 0
Changed lines of the file:
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@@
     (pad_size 3.5 3.5)
     (pad_drill 2)
-    (pad_to_mask_clearance 0.05)
+    (pad_to_mask_clearance 0)
     (aux_axis_origin 0 0)
     (grid_origin 160 190)
@@
   (module SFUSat:MOLEX_FFC-14 (layer F.Cu)
     (at 160 312.01)
+    (solder_mask_margin 0.02)
     (fp_text reference J9 (at -6.5 1.6) (layer F.SilkS) hide
       (effects (font (size 1 1) (thickness 0.15)))
@@
   (module SFUSat:MOLEX_FFC-14 (layer F.Cu)
     (at 160 50.16 180)
+    (solder_mask_margin 0.02)
     (fp_text reference J10 (at -5.5 0.16 270) (layer F.SilkS)
       (effects (font (size 1 1) (thickness 0.15)))
@@
   (module SFUSat:MOLEX_FFC-14 (layer F.Cu)
     (at 160 316.17)
+    (solder_mask_margin 0.02)
     (fp_text reference J3 (at -2.25 -1.5) (layer F.SilkS) hide
       (effects (font (size 1 1) (thickness 0.15)))
@@
   (module SFUSat:VSSOP_8 (layer F.Cu)
     (at 196.6 182.8 90)
+    (solder_mask_margin 0.02)
     (fp_text reference U5 (at -2.6 -2.2 180) (layer F.SilkS)
       (effects (font (size 1 1) (thickness 0.15)))
@@
   (module SFUSat:VSSOP_8 (layer F.Cu)
     (at 134.639998 328.55)
+    (solder_mask_margin 0.02)
     (fp_text reference U3 (at -2.439998 -1.95 180) (layer F.SilkS)
       (effects (font (size 1 1) (thickness 0.15)))
@@
   (module SFUSat:VSSOP_8 (layer F.Cu)
     (at 123.4 74.6 270)
+    (solder_mask_margin 0.02)
     (fp_text reference U1 (at -2.6 -2.2 360) (layer F.SilkS)
       (effects (font (size 1 1) (thickness 0.15)))
@@
   (module SFUSat:VSSOP_8 (layer F.Cu)
     (at 123.4 183 90)
+    (solder_mask_margin 0.02)
     (fp_text reference U2 (at -2.8 -2 180) (layer F.SilkS)
       (effects (font (size 1 1) (thickness 0.15)))
@@
   (module SFUSat:VSSOP_8 (layer F.Cu)
     (at 196.25 74.85 270)
+    (solder_mask_margin 0.02)
     (fp_text reference U4 (at -2.65 -2.35 360) (layer F.SilkS)
       (effects (font (size 1 1) (thickness 0.15)))
@@
   (module SFUSat:VSSOP_8 (layer F.Cu)
     (at 187.7 328.6 180)
+    (solder_mask_margin 0.02)
     (fp_text reference U6 (at -0.5 4 360) (layer F.SilkS)
       (effects (font (size 1 1) (thickness 0.15)))

Commit message: rev 2 done
Parts:
- moved P1 1.00 mm to (140.0, 57.5)
- moved P7 1.00 mm to (180.0, 57.5)
Routing:
- net /PV1+: track 301.0 -> 295.5 mm
- net /DA: track 289.8 -> 287.5 mm
- net Net-(P7-Pad2): track 74.3 -> 75.9 mm
- net /DB: track 288.6 -> 287.1 mm
Other:
- outline, holes or cut-outs redrawn
- board text added: "SFU Satellite Design Team Panel Rev. 2"
- board text removed: "SFU Satellite Design Team Panel Rev. 1"
